Commit message: Implemented speed and position control, static friction id

File: exo_right_arm_ws/install/exo_description/share/exo_description/urdf/exo.xacro (robot description, xacro)
@@ -169,4 +169,5 @@
   <child link="Motor1_1"/>
   <axis xyz="-1.0 -0.0 0.0"/>
+  <dynamics damping="0.012" friction="0.1184"/>
 </joint>
 <joint name="Rigid 2" type="fixed">
@@ -185,4 +186,5 @@
   <child link="Componente3_v1_1"/>
   <axis xyz="-0.0 1.0 -0.0"/>
+  <dynamics damping="0.012" friction="0.1184"/>
 </joint>
 <joint name="Rigid 6" type="fixed">
@@ -196,4 +198,5 @@
   <child link="Motor3_1"/>
   <axis xyz="-0.0 -1.0 -0.0"/>
+  <dynamics damping="0.012" friction="0.1184"/>
 </joint>
 <joint name="Rigid 8" type="fixed">
@@ -210,5 +213,5 @@
     <state_interface name="position"/>
     <state_interface name="velocity"/>
-    <state_interface name="torque"/>
+    <state_interface name="effort"/>
   </joint>
   <joint name="Revolute 5">
@@ -216,5 +219,5 @@
     <state_interface name="position"/>
     <state_interface name="velocity"/>
-    <state_interface name="torque"/>
+    <state_interface name="effort"/>
   </joint>
   <joint name="Revolute 7">
@@ -222,5 +225,5 @@
     <state_interface name="position"/>
     <state_interface name="velocity"/>
-    <state_interface name="torque"/>
+    <state_interface name="effort"/>
   </joint>
 </ros2_control>

File: exo_right_arm_ws/src/install/exo_description/share/exo_description/urdf/exo.xacro (robot description, xacro)
@@ -210,5 +210,5 @@
     <state_interface name="position"/>
     <state_interface name="velocity"/>
-    <state_interface name="torque"/>
+    <state_interface name="effort"/>
   </joint>
   <joint name="Revolute 5">
@@ -216,5 +216,5 @@
     <state_interface name="position"/>
     <state_interface name="velocity"/>
-    <state_interface name="torque"/>
+    <state_interface name="effort"/>
   </joint>
   <joint name="Revolute 7">
@@ -222,5 +222,5 @@
     <state_interface name="position"/>
     <state_interface name="velocity"/>
-    <state_interface name="torque"/>
+    <state_interface name="effort"/>
   </joint>
 </ros2_control>

Commit message: renamed joints

File: exo_right_arm_ws/install/exo_description/share/exo_description/urdf/exo.xacro (robot description, xacro)
@@ -164,5 +164,5 @@
   </collision>
 </link>
-<joint name="Revolute 1" type="continuous">
+<joint name="revolute_1" type="continuous">
   <origin xyz="-0.014 0.0 0.0" rpy="0 0 0"/>
   <parent link="base_link"/>
@@ -181,5 +181,5 @@
   <child link="Motor2_1"/>
 </joint>
-<joint name="Revolute 5" type="continuous">
+<joint name="revolute_2" type="continuous">
   <origin xyz="0.0 0.003 0.0" rpy="0 0 0"/>
   <parent link="Motor2_1"/>
@@ -193,5 +193,5 @@
   <child link="Componente4_v1_1"/>
 </joint>
-<joint name="Revolute 7" type="continuous">
+<joint name="revolute_3" type="continuous">
   <origin xyz="0.002653 -0.0095 -0.24002" rpy="0 0 0"/>
   <parent link="Componente4_v1_1"/>
@@ -205,9 +205,15 @@
   <child link="Componente5_v1_1"/>
 </joint>
+<xacro:arg name="hardware" default="real"/>
 <ros2_control name="exo_right_arm" type="system">
   <hardware>
-    <plugin>exo_hardware/teensy_plugin</plugin>
+    <xacro:if value="${hardware == 'real'}">
+      <plugin>exo_hardware/teensy_plugin</plugin>
+    </xacro:if>
+    <xacro:if value="${hardware == 'gazebo'}">
+      <plugin>gazebo_ros2_control/GazeboSystem</plugin>
+    </xacro:if>
   </hardware>
-  <joint name="Revolute 1">
+  <joint name="revolute_1">
     <command_interface name="effort"/>
     <state_interface name="position"/>
@@ -215,5 +221,5 @@
     <state_interface name="effort"/>
   </joint>
-  <joint name="Revolute 5">
+  <joint name="revolute_2">
     <command_interface name="effort"/>
     <state_interface name="position"/>
@@ -221,5 +227,5 @@
     <state_interface name="effort"/>
   </joint>
-  <joint name="Revolute 7">
+  <joint name="revolute_3">
     <command_interface name="effort"/>
     <state_interface name="position"/>

File: exo_right_arm_ws/src/install/exo_description/share/exo_description/urdf/exo.xacro (robot description, xacro)
@@ -164,5 +164,5 @@
   </collision>
 </link>
-<joint name="Revolute 1" type="continuous">
+<joint name="revolute_1" type="continuous">
   <origin xyz="-0.014 0.0 0.0" rpy="0 0 0"/>
   <parent link="base_link"/>
@@ -180,5 +180,5 @@
   <child link="Motor2_1"/>
 </joint>
-<joint name="Revolute 5" type="continuous">
+<joint name="revolute_5" type="continuous">
   <origin xyz="0.0 0.003 0.0" rpy="0 0 0"/>
   <parent link="Motor2_1"/>
@@ -191,5 +191,5 @@
   <child link="Componente4_v1_1"/>
 </joint>
-<joint name="Revolute 7" type="continuous">
+<joint name="revolute_7" type="continuous">
   <origin xyz="0.002653 -0.0095 -0.24002" rpy="0 0 0"/>
   <parent link="Componente4_v1_1"/>
@@ -206,5 +206,5 @@
     <plugin>exo_hardware/teensy_plugin</plugin>
   </hardware>
-  <joint name="Revolute 1">
+  <joint name="revolute_1">
     <command_interface name="effort"/>
     <state_interface name="position"/>
@@ -212,5 +212,5 @@
     <state_interface name="effort"/>
   </joint>
-  <joint name="Revolute 5">
+  <joint name="revolute_5">
     <command_interface name="effort"/>
     <state_interface name="position"/>
@@ -218,5 +218,5 @@
     <state_interface name="effort"/>
   </joint>
-  <joint name="Revolute 7">
+  <joint name="revolute_7">
     <command_interface name="effort"/>
     <state_interface name="position"/>

Commit message: rviz

File: exo_right_arm_ws/install/exo_description/share/exo_description/urdf/exo.xacro (robot description, xacro)
@@ -4,4 +4,10 @@
 <xacro:include filename="$(find exo_description)/urdf/exo.trans" />
 <xacro:include filename="$(find exo_description)/urdf/exo.gazebo" />
+<link name="base"/>
+<joint name="base_to_base_link" type="fixed">
+  <parent link="base"/>
+  <child link="base_link"/>
+  <origin xyz="0 0 0" rpy="0 0 0"/>
+</joint>
 <link name="base_link">
   <inertial>
@@ -171,10 +177,10 @@
   <dynamics damping="0.012" friction="0.1184"/>
 </joint>
-<joint name="Rigid 2" type="fixed">
+<joint name="rigid_2" type="fixed">
   <origin xyz="-0.003 0.0 0.0" rpy="0 0 0"/>
   <parent link="Motor1_1"/>
   <child link="Componente2_v1_1"/>
 </joint>
-<joint name="Rigid 3" type="fixed">
+<joint name="rigid_3" type="fixed">
   <origin xyz="0.087 -0.087 0.0" rpy="0 0 0"/>
   <parent link="Componente2_v1_1"/>
@@ -188,5 +194,5 @@
   <dynamics damping="0.012" friction="0.1184"/>
 </joint>
-<joint name="Rigid 6" type="fixed">
+<joint name="rigid_6" type="fixed">
   <origin xyz="0.00033 0.003 -0.045569" rpy="0 0 0"/>
   <parent link="Componente3_v1_1"/>
@@ -200,5 +206,5 @@
   <dynamics damping="0.012" friction="0.1184"/>
 </joint>
-<joint name="Rigid 8" type="fixed">
+<joint name="rigid_8" type="fixed">
   <origin xyz="0.0 -0.003 0.0" rpy="0 0 0"/>
   <parent link="Motor3_1"/>
@@ -208,8 +214,8 @@
 <ros2_control name="exo_right_arm" type="system">
   <hardware>
-    <xacro:if value="${hardware == 'real'}">
+    <xacro:if value="${xacro.arg('hardware') == 'real'}">
       <plugin>exo_hardware/teensy_plugin</plugin>
     </xacro:if>
-    <xacro:if value="${hardware == 'gazebo'}">
+    <xacro:if value="${xacro.arg('hardware') == 'gazebo'}">
       <plugin>gazebo_ros2_control/GazeboSystem</plugin>
     </xacro:if>

File: exo_right_arm_ws/src/install/exo_description/share/exo_description/urdf/exo.xacro (robot description, xacro)
@@ -170,10 +170,10 @@
   <axis xyz="-1.0 -0.0 0.0"/>
 </joint>
-<joint name="Rigid 2" type="fixed">
+<joint name="rigid_2" type="fixed">
   <origin xyz="-0.003 0.0 0.0" rpy="0 0 0"/>
   <parent link="Motor1_1"/>
   <child link="Componente2_v1_1"/>
 </joint>
-<joint name="Rigid 3" type="fixed">
+<joint name="rigid_3" type="fixed">
   <origin xyz="0.087 -0.087 0.0" rpy="0 0 0"/>
   <parent link="Componente2_v1_1"/>
@@ -186,5 +186,5 @@
   <axis xyz="-0.0 1.0 -0.0"/>
 </joint>
-<joint name="Rigid 6" type="fixed">
+<joint name="rigid_6" type="fixed">
   <origin xyz="0.00033 0.003 -0.045569" rpy="0 0 0"/>
   <parent link="Componente3_v1_1"/>
@@ -197,5 +197,5 @@
   <axis xyz="-0.0 -1.0 -0.0"/>
 </joint>
-<joint name="Rigid 8" type="fixed">
+<joint name="rigid_8" type="fixed">
   <origin xyz="0.0 -0.003 0.0" rpy="0 0 0"/>
   <parent link="Motor3_1"/>

Commit message: gazebo and first controller implemented

File: exo_right_arm_ws/install/exo_description/share/exo_description/urdf/exo.xacro (robot description, xacro)
@@ -1,12 +1,13 @@
 <?xml version="1.0" ?>
 <robot name="exo" xmlns:xacro="http://www.ros.org/wiki/xacro">
+<xacro:arg name="hardware" default="real"/>
+<xacro:arg name="controller_config" default="controllers_effort.yaml"/>
 <xacro:include filename="$(find exo_description)/urdf/materials.xacro" />
 <xacro:include filename="$(find exo_description)/urdf/exo.trans" />
-<xacro:include filename="$(find exo_description)/urdf/exo.gazebo" />
-<link name="base"/>
-<joint name="base_to_base_link" type="fixed">
-  <parent link="base"/>
+<link name="world"/>
+<joint name="world_fixed" type="fixed">
+  <parent link="world"/>
   <child link="base_link"/>
-  <origin xyz="0 0 0" rpy="0 0 0"/>
+  <origin xyz="0 0 0.6" rpy="0 0 0"/>
 </joint>
 <link name="base_link">
@@ -41,5 +42,5 @@
       <mesh filename="package://exo_description/meshes/Motor1_1.stl" scale="0.001 0.001 0.001"/>
     </geometry>
-    <material name="silver"/>
+    <material name="black"/>
   </visual>
   <collision>
@@ -81,5 +82,5 @@
       <mesh filename="package://exo_description/meshes/Motor2_1.stl" scale="0.001 0.001 0.001"/>
     </geometry>
-    <material name="silver"/>
+    <material name="black"/>
   </visual>
   <collision>
@@ -141,5 +142,5 @@
       <mesh filename="package://exo_description/meshes/Motor3_1.stl" scale="0.001 0.001 0.001"/>
     </geometry>
-    <material name="silver"/>
+    <material name="black"/>
   </visual>
   <collision>
@@ -170,5 +171,5 @@
   </collision>
 </link>
-<joint name="revolute_1" type="continuous">
+<joint name="revolute_1" type="revolute">
   <origin xyz="-0.014 0.0 0.0" rpy="0 0 0"/>
   <parent link="base_link"/>
@@ -176,4 +177,5 @@
   <axis xyz="-1.0 -0.0 0.0"/>
   <dynamics damping="0.012" friction="0.1184"/>
+  <limit lower="0" upper="1.919" effort="20" velocity="11"/>
 </joint>
 <joint name="rigid_2" type="fixed">
@@ -187,10 +189,11 @@
   <child link="Motor2_1"/>
 </joint>
-<joint name="revolute_2" type="continuous">
+<joint name="revolute_2" type="revolute">
   <origin xyz="0.0 0.003 0.0" rpy="0 0 0"/>
   <parent link="Motor2_1"/>
   <child link="Componente3_v1_1"/>
-  <axis xyz="-0.0 1.0 -0.0"/>
+  <axis xyz="0.0 -1.0 0.0"/>
   <dynamics damping="0.012" friction="0.1184"/>
+  <limit lower="-0.56" upper="2.793" effort="20" velocity="11"/>
 </joint>
 <joint name="rigid_6" type="fixed">
@@ -199,5 +202,5 @@
   <child link="Componente4_v1_1"/>
 </joint>
-<joint name="revolute_3" type="continuous">
+<joint name="revolute_3" type="revolute">
   <origin xyz="0.002653 -0.0095 -0.24002" rpy="0 0 0"/>
   <parent link="Componente4_v1_1"/>
@@ -205,4 +208,5 @@
   <axis xyz="-0.0 -1.0 -0.0"/>
   <dynamics damping="0.012" friction="0.1184"/>
+  <limit lower="0" upper="2.094" effort="20" velocity="11"/>
 </joint>
 <joint name="rigid_8" type="fixed">
@@ -211,5 +215,4 @@
   <child link="Componente5_v1_1"/>
 </joint>
-<xacro:arg name="hardware" default="real"/>
 <ros2_control name="exo_right_arm" type="system">
   <hardware>
@@ -218,5 +221,5 @@
     </xacro:if>
     <xacro:if value="${xacro.arg('hardware') == 'gazebo'}">
-      <plugin>gazebo_ros2_control/GazeboSystem</plugin>
+      <plugin>gz_ros2_control/GazeboSimSystem</plugin>
     </xacro:if>
   </hardware>
@@ -240,3 +243,6 @@
   </joint>
 </ros2_control>
+<xacro:if value="${xacro.arg('hardware') == 'gazebo'}">
+  <xacro:include filename="$(find exo_description)/urdf/exo.gazebo"/>
+</xacro:if>
 </robot>

File: exo_right_arm_ws/install/exo_description/share/exo_description/urdf/materials.xacro (robot description, xacro)
@@ -4,3 +4,6 @@
   <color rgba="0.700 0.700 0.700 1.000"/>
 </material>
+<material name="black">
+  <color rgba="0.200 0.200 0.200 1.000"/>
+</material>
 </robot>

Commit message: Update environment setup script and egg-info sources; remove install log. Added new environment variables for Terminator and updated PYTHONPATH. Adjusted SOURCES.txt to reflect new file structure and included additional configuration files.

File: exo_right_arm_ws/install/exo_description/share/exo_description/urdf/exo.xacro (robot description, xacro)
@@ -1,248 +1 @@
-<?xml version="1.0" ?>
-<robot name="exo" xmlns:xacro="http://www.ros.org/wiki/xacro">
-<xacro:arg name="hardware" default="real"/>
-<xacro:arg name="controller_config" default="controllers_effort.yaml"/>
-<xacro:include filename="$(find exo_description)/urdf/materials.xacro" />
-<xacro:include filename="$(find exo_description)/urdf/exo.trans" />
-<link name="world"/>
-<joint name="world_fixed" type="fixed">
-  <parent link="world"/>
-  <child link="base_link"/>
-  <origin xyz="0 0 0.6" rpy="0 0 0"/>
-</joint>
-<link name="base_link">
-  <inertial>
-    <origin xyz="0.012748850487473646 0.0012395946054243722 0.013826907905998666" rpy="0 0 0"/>
-    <mass value="0.07388024509698206"/>
-    <inertia ixx="8e-05" iyy="0.000154" izz="0.000109" ixy="2e-06" iyz="-1e-05" ixz="-5.1e-05"/>
-  </inertial>
-  <visual>
-    <origin xyz="0 0 0" rpy="0 0 0"/>
-    <geometry>
-      <mesh filename="package://exo_description/meshes/base_link.stl" scale="0.001 0.001 0.001"/>
-    </geometry>
-    <material name="silver"/>
-  </visual>
-  <collision>
-    <origin xyz="0 0 0" rpy="0 0 0"/>
-    <geometry>
-      <mesh filename="package://exo_description/meshes/base_link.stl" scale="0.001 0.001 0.001"/>
-    </geometry>
-  </collision>
-</link>
-<link name="Motor1_1">
-  <inertial>
-    <origin xyz="-0.02865689684955547 0.0008019947900518482 -0.00013732170892716988" rpy="0 0 0"/>
-    <mass value="0.33655764736226634"/>
-    <inertia ixx="0.000158" iyy="0.000206" izz="0.000208" ixy="7e-06" iyz="-0.0" ixz="-1e-06"/>
-  </inertial>
-  <visual>
-    <origin xyz="0.014 0.0 -0.0" rpy="0 0 0"/>
-    <geometry>
-      <mesh filename="package://exo_description/meshes/Motor1_1.stl" scale="0.001 0.001 0.001"/>
-    </geometry>
-    <material name="black"/>
-  </visual>
-  <collision>
-    <origin xyz="0.014 0.0 -0.0" rpy="0 0 0"/>
-    <geometry>
-      <mesh filename="package://exo_description/meshes/Motor1_1.stl" scale="0.001 0.001 0.001"/>
-    </geometry>
-  </collision>
-</link>
-<link name="Componente2_v1_1">
-  <inertial>
-    <origin xyz="0.025697121565106763 -0.06800197164371612 0.0006322543327434366" rpy="0 0 0"/>
-    <mass value="0.0856142757419247"/>
-    <inertia ixx="0.000127" iyy="0.000133" izz="0.000214" ixy="6.9e-05" iyz="1e-06" ixz="-6e-06"/>
-  </inertial>
-  <visual>
-    <origin xyz="0.017 0.0 -0.0" rpy="0 0 0"/>
-    <geometry>
-      <mesh filename="package://exo_description/meshes/Componente2_v1_1.stl" scale="0.001 0.001 0.001"/>
-    </geometry>
-    <material name="silver"/>
-  </visual>
-  <collision>
-    <origin xyz="0.017 0.0 -0.0" rpy="0 0 0"/>
-    <geometry>
-      <mesh filename="package://exo_description/meshes/Componente2_v1_1.stl" scale="0.001 0.001 0.001"/>
-    </geometry>
-  </collision>
-</link>
-<link name="Motor2_1">
-  <inertial>
-    <origin xyz="0.0008019947900903546 -0.025656896849592187 0.00013732170895816803" rpy="0 0 0"/>
-    <mass value="0.33655764736226634"/>
-    <inertia ixx="0.000206" iyy="0.000158" izz="0.000208" ixy="7e-06" iyz="1e-06" ixz="0.0"/>
-  </inertial>
-  <visual>
-    <origin xyz="-0.07 0.087 -0.0" rpy="0 0 0"/>
-    <geometry>
-      <mesh filename="package://exo_description/meshes/Motor2_1.stl" scale="0.001 0.001 0.001"/>
-    </geometry>
-    <material name="black"/>
-  </visual>
-  <collision>
-    <origin xyz="-0.07 0.087 -0.0" rpy="0 0 0"/>
-    <geometry>
-      <mesh filename="package://exo_description/meshes/Motor2_1.stl" scale="0.001 0.001 0.001"/>
-    </geometry>
-  </collision>
-</link>
-<link name="Componente3_v1_1">
-  <inertial>
-    <origin xyz="0.00032953390008541583 0.004560809428740015 -0.04548170531617862" rpy="0 0 0"/>
-    <mass value="0.02436487236137751"/>
-    <inertia ixx="4.5e-05" iyy="4.7e-05" izz="3e-06" ixy="-0.0" iyz="0.0" ixz="0.0"/>
-  </inertial>
-  <visual>
-    <origin xyz="-0.07 0.084 -0.0" rpy="0 0 0"/>
-    <geometry>
-      <mesh filename="package://exo_description/meshes/Componente3_v1_1.stl" scale="0.001 0.001 0.001"/>
-    </geometry>
-    <material name="silver"/>
-  </visual>
-  <collision>
-    <origin xyz="-0.07 0.084 -0.0" rpy="0 0 0"/>
-    <geometry>
-      <mesh filename="package://exo_description/meshes/Componente3_v1_1.stl" scale="0.001 0.001 0.001"/>
-    </geometry>
-  </collision>
-</link>
-<link name="Componente4_v1_1">
-  <inertial>
-    <origin xyz="-0.010220970902704345 0.012182176440413015 -0.11338415880449806" rpy="0 0 0"/>
-    <mass value="0.16326913907635673"/>
-    <inertia ixx="0.000882" iyy="0.000951" izz="0.000135" ixy="3.1e-05" iyz="-4.9e-05" ixz="-3.5e-05"/>
-  </inertial>
-  <visual>
-    <origin xyz="-0.07033 0.081 0.045569" rpy="0 0 0"/>
-    <geometry>
-      <mesh filename="package://exo_description/meshes/Componente4_v1_1.stl" scale="0.001 0.001 0.001"/>
-    </geometry>
-    <material name="silver"/>
-  </visual>
-  <collision>
-    <origin xyz="-0.07033 0.081 0.045569" rpy="0 0 0"/>
-    <geometry>
-      <mesh filename="package://exo_description/meshes/Componente4_v1_1.stl" scale="0.001 0.001 0.001"/>
-    </geometry>
-  </collision>
-</link>
-<link name="Motor3_1">
-  <inertial>
-    <origin xyz="0.0005883974851695895 -0.028656896849589955 0.0005618260705803624" rpy="0 0 0"/>
-    <mass value="0.33655764736226634"/>
-    <inertia ixx="0.000207" iyy="0.000158" izz="0.000208" ixy="5e-06" iyz="5e-06" ixz="-1e-06"/>
-  </inertial>
-  <visual>
-    <origin xyz="-0.072983 0.0905 0.285589" rpy="0 0 0"/>
-    <geometry>
-      <mesh filename="package://exo_description/meshes/Motor3_1.stl" scale="0.001 0.001 0.001"/>
-    </geometry>
-    <material name="black"/>
-  </visual>
-  <collision>
-    <origin xyz="-0.072983 0.0905 0.285589" rpy="0 0 0"/>
-    <geometry>
-      <mesh filename="package://exo_description/meshes/Motor3_1.stl" scale="0.001 0.001 0.001"/>
-    </geometry>
-  </collision>
-</link>
-<link name="Componente5_v1_1">
-  <inertial>
-    <origin xyz="-0.012433445660119731 0.009030253916196301 -0.08353720706436124" rpy="0 0 0"/>
-    <mass value="0.07092422473137162"/>
-    <inertia ixx="0.000201" iyy="0.000217" izz="4.3e-05" ixy="1.4e-05" iyz="1.9e-05" ixz="-1.7e-05"/>
-  </inertial>
-  <visual>
-    <origin xyz="-0.072983 0.0935 0.285589" rpy="0 0 0"/>
-    <geometry>
-      <mesh filename="package://exo_description/meshes/Componente5_v1_1.stl" scale="0.001 0.001 0.001"/>
-    </geometry>
-    <material name="silver"/>
-  </visual>
-  <collision>
-    <origin xyz="-0.072983 0.0935 0.285589" rpy="0 0 0"/>
-    <geometry>
-      <mesh filename="package://exo_description/meshes/Componente5_v1_1.stl" scale="0.001 0.001 0.001"/>
-    </geometry>
-  </collision>
-</link>
-<joint name="revolute_1" type="revolute">
-  <origin xyz="-0.014 0.0 0.0" rpy="0 0 0"/>
-  <parent link="base_link"/>
-  <child link="Motor1_1"/>
-  <axis xyz="-1.0 -0.0 0.0"/>
-  <dynamics damping="0.012" friction="0.1184"/>
-  <limit lower="0" upper="1.919" effort="20" velocity="11"/>
-</joint>
-<joint name="rigid_2" type="fixed">
-  <origin xyz="-0.003 0.0 0.0" rpy="0 0 0"/>
-  <parent link="Motor1_1"/>
-  <child link="Componente2_v1_1"/>
-</joint>
-<joint name="rigid_3" type="fixed">
-  <origin xyz="0.087 -0.087 0.0" rpy="0 0 0"/>
-  <parent link="Componente2_v1_1"/>
-  <child link="Motor2_1"/>
-</joint>
-<joint name="revolute_2" type="revolute">
-  <origin xyz="0.0 0.003 0.0" rpy="0 0 0"/>
-  <parent link="Motor2_1"/>
-  <child link="Componente3_v1_1"/>
-  <axis xyz="0.0 -1.0 0.0"/>
-  <dynamics damping="0.012" friction="0.1184"/>
-  <limit lower="-0.56" upper="2.793" effort="20" velocity="11"/>
-</joint>
-<joint name="rigid_6" type="fixed">
-  <origin xyz="0.00033 0.003 -0.045569" rpy="0 0 0"/>
-  <parent link="Componente3_v1_1"/>
-  <child link="Componente4_v1_1"/>
-</joint>
-<joint name="revolute_3" type="revolute">
-  <origin xyz="0.002653 -0.0095 -0.24002" rpy="0 0 0"/>
-  <parent link="Componente4_v1_1"/>
-  <child link="Motor3_1"/>
-  <axis xyz="-0.0 -1.0 -0.0"/>
-  <dynamics damping="0.012" friction="0.1184"/>
-  <limit lower="0" upper="2.094" effort="20" velocity="11"/>
-</joint>
-<joint name="rigid_8" type="fixed">
-  <origin xyz="0.0 -0.003 0.0" rpy="0 0 0"/>
-  <parent link="Motor3_1"/>
-  <child link="Componente5_v1_1"/>
-</joint>
-<ros2_control name="exo_right_arm" type="system">
-  <hardware>
-    <xacro:if value="${xacro.arg('hardware') == 'real'}">
-      <plugin>exo_hardware/teensy_plugin</plugin>
-    </xacro:if>
-    <xacro:if value="${xacro.arg('hardware') == 'gazebo'}">
-      <plugin>gz_ros2_control/GazeboSimSystem</plugin>
-    </xacro:if>
-  </hardware>
-  <joint name="revolute_1">
-    <command_interface name="effort"/>
-    <state_interface name="position"/>
-    <state_interface name="velocity"/>
-    <state_interface name="effort"/>
-  </joint>
-  <joint name="revolute_2">
-    <command_interface name="effort"/>
-    <state_interface name="position"/>
-    <state_interface name="velocity"/>
-    <state_interface name="effort"/>
-  </joint>
-  <joint name="revolute_3">
-    <command_interface name="effort"/>
-    <state_interface name="position"/>
-    <state_interface name="velocity"/>
-    <state_interface name="effort"/>
-  </joint>
-</ros2_control>
-<xacro:if value="${xacro.arg('hardware') == 'gazebo'}">
-  <xacro:include filename="$(find exo_description)/urdf/exo.gazebo"/>
-</xacro:if>
-</robot>
+/home/farid/tesis/exo_right_arm_ws/src/exo_description/urdf/exo.xacro

File: exo_right_arm_ws/install/exo_description/share/exo_description/urdf/materials.xacro (robot description, xacro)
@@ -1,9 +1 @@
-<?xml version="1.0" ?>
-<robot name="RightArm" xmlns:xacro="http://www.ros.org/wiki/xacro" >
-<material name="silver">
-  <color rgba="0.700 0.700 0.700 1.000"/>
-</material>
-<material name="black">
-  <color rgba="0.200 0.200 0.200 1.000"/>
-</material>
-</robot>
+/home/farid/tesis/exo_right_arm_ws/src/exo_description/urdf/materials.xacro
