Commit message: fixed single arm issues

File: exo_right_arm_ws/src/exo_description/urdf/exo.xacro (robot description, xacro)
@@ -2,6 +2,8 @@
 <robot name="exo" xmlns:xacro="http://www.ros.org/wiki/xacro">
 <xacro:arg name="hardware" default="real"/>
-<xacro:arg name="controller_config" default="controllers_effort.yaml"/>
-<!-- arms: right (default), left, or dual. Single-arm modes use unprefixed joints. -->
+<!-- Per-arm controller YAML files passed to gz_ros2_control. Either may be empty. -->
+<xacro:arg name="controller_config_left" default=""/>
+<xacro:arg name="controller_config_right" default=""/>
+<!-- arms: right (default), left, or dual. All three modes use prefixed joints. -->
 <xacro:arg name="arms" default="right"/>
 <!-- Optional fixed mounts (base_link) for each arm in dual mode (meters, radians). -->
@@ -27,26 +29,21 @@
   <origin xyz="0 0 0.6" rpy="0 0 0"/>
 </joint>
-<xacro:if value="${xacro.arg('arms') == 'dual'}">
-  <link name="base_link">
-    <inertial>
-      <origin xyz="0 0 0" rpy="0 0 0"/>
-      <mass value="0.001"/>
-      <inertia ixx="1e-06" iyy="1e-06" izz="1e-06" ixy="0" iyz="0" ixz="0"/>
-    </inertial>
-  </link>
-</xacro:if>
-<xacro:if value="${xacro.arg('arms') == 'dual'}">
+<!-- All modes mount each arm under a shared base_link with prefix-aware mount joints. -->
+<link name="base_link">
+  <inertial>
+    <origin xyz="0 0 0" rpy="0 0 0"/>
+    <mass value="0.001"/>
+    <inertia ixx="1e-06" iyy="1e-06" izz="1e-06" ixy="0" iyz="0" ixz="0"/>
+  </inertial>
+</link>
+<xacro:if value="${xacro.arg('arms') == 'dual' or xacro.arg('arms') == 'right'}">
   <xacro:exo_arm_right prefix="right_"
     mount_x="${xacro.arg('right_mount_x')}" mount_y="${xacro.arg('right_mount_y')}" mount_z="${xacro.arg('right_mount_z')}"
     mount_roll="${xacro.arg('right_mount_roll')}" mount_pitch="${xacro.arg('right_mount_pitch')}" mount_yaw="${xacro.arg('right_mount_yaw')}"/>
+</xacro:if>
+<xacro:if value="${xacro.arg('arms') == 'dual' or xacro.arg('arms') == 'left'}">
   <xacro:exo_arm_left prefix="left_"
     mount_x="${xacro.arg('left_mount_x')}" mount_y="${xacro.arg('left_mount_y')}" mount_z="${xacro.arg('left_mount_z')}"
     mount_roll="${xacro.arg('left_mount_roll')}" mount_pitch="${xacro.arg('left_mount_pitch')}" mount_yaw="${xacro.arg('left_mount_yaw')}"/>
-</xacro:if>
-<xacro:if value="${xacro.arg('arms') == 'right'}">
-  <xacro:exo_arm_right prefix="" mount_x="0" mount_y="0" mount_z="0" mount_roll="0" mount_pitch="0" mount_yaw="0"/>
-</xacro:if>
-<xacro:if value="${xacro.arg('arms') == 'left'}">
-  <xacro:exo_arm_left prefix="" mount_x="0" mount_y="0" mount_z="0" mount_roll="0" mount_pitch="0" mount_yaw="0"/>
 </xacro:if>
 <ros2_control name="exo_system" type="system">
@@ -76,5 +73,6 @@
     </xacro:if>
   </hardware>
-  <xacro:if value="${xacro.arg('arms') == 'dual'}">
+  <!-- Joint declarations: always prefixed (right_/left_), so all arm modes use the same naming. -->
+  <xacro:if value="${xacro.arg('arms') == 'dual' or xacro.arg('arms') == 'right'}">
     <joint name="right_revolute_1">
       <command_interface name="effort"/>
@@ -95,4 +93,6 @@
       <state_interface name="effort"/>
     </joint>
+  </xacro:if>
+  <xacro:if value="${xacro.arg('arms') == 'dual' or xacro.arg('arms') == 'left'}">
     <joint name="left_revolute_1">
       <command_interface name="effort"/>
@@ -114,24 +114,4 @@
     </joint>
   </xacro:if>
-  <xacro:unless value="${xacro.arg('arms') == 'dual'}">
-    <joint name="revolute_1">
-      <command_interface name="effort"/>
-      <state_interface name="position"/>
-      <state_interface name="velocity"/>
-      <state_interface name="effort"/>
-    </joint>
-    <joint name="revolute_2">
-      <command_interface name="effort"/>
-      <state_interface name="position"/>
-      <state_interface name="velocity"/>
-      <state_interface name="effort"/>
-    </joint>
-    <joint name="revolute_3">
-      <command_interface name="effort"/>
-      <state_interface name="position"/>
-      <state_interface name="velocity"/>
-      <state_interface name="effort"/>
-    </joint>
-  </xacro:unless>
 </ros2_control>
 <xacro:if value="${xacro.arg('hardware') == 'gazebo'}">

Commit message: exo_description update and smc tuning

File: exo_right_arm_ws/src/exo_description/urdf/exo.xacro (robot description, xacro)
@@ -7,4 +7,6 @@
 <!-- arms: right (default), left, or dual. All three modes use prefixed joints. -->
 <xacro:arg name="arms" default="right"/>
+<!-- Set to true to include collision geometry and joint friction/damping (simulation only). -->
+<xacro:arg name="joint_dynamics" default="false"/>
 <!-- Optional fixed mounts (base_link) for each arm in dual mode (meters, radians). -->
 <xacro:arg name="right_mount_x" default="0"/>
@@ -40,10 +42,12 @@
   <xacro:exo_arm_right prefix="right_"
     mount_x="${xacro.arg('right_mount_x')}" mount_y="${xacro.arg('right_mount_y')}" mount_z="${xacro.arg('right_mount_z')}"
-    mount_roll="${xacro.arg('right_mount_roll')}" mount_pitch="${xacro.arg('right_mount_pitch')}" mount_yaw="${xacro.arg('right_mount_yaw')}"/>
+    mount_roll="${xacro.arg('right_mount_roll')}" mount_pitch="${xacro.arg('right_mount_pitch')}" mount_yaw="${xacro.arg('right_mount_yaw')}"
+    joint_dynamics="${xacro.arg('joint_dynamics')}"/>
 </xacro:if>
 <xacro:if value="${xacro.arg('arms') == 'dual' or xacro.arg('arms') == 'left'}">
   <xacro:exo_arm_left prefix="left_"
     mount_x="${xacro.arg('left_mount_x')}" mount_y="${xacro.arg('left_mount_y')}" mount_z="${xacro.arg('left_mount_z')}"
-    mount_roll="${xacro.arg('left_mount_roll')}" mount_pitch="${xacro.arg('left_mount_pitch')}" mount_yaw="${xacro.arg('left_mount_yaw')}"/>
+    mount_roll="${xacro.arg('left_mount_roll')}" mount_pitch="${xacro.arg('left_mount_pitch')}" mount_yaw="${xacro.arg('left_mount_yaw')}"
+    joint_dynamics="${xacro.arg('joint_dynamics')}"/>
 </xacro:if>
 <ros2_control name="exo_system" type="system">
@@ -77,5 +81,7 @@
     <joint name="right_revolute_1">
       <command_interface name="effort"/>
-      <state_interface name="position"/>
+      <state_interface name="position">
+        <param name="initial_value">-1.53</param>
+      </state_interface>
       <state_interface name="velocity"/>
       <state_interface name="effort"/>
@@ -83,5 +89,7 @@
     <joint name="right_revolute_2">
       <command_interface name="effort"/>
-      <state_interface name="position"/>
+      <state_interface name="position">
+        <param name="initial_value">-2.82</param>
+      </state_interface>
       <state_interface name="velocity"/>
       <state_interface name="effort"/>
@@ -89,5 +97,7 @@
     <joint name="right_revolute_3">
       <command_interface name="effort"/>
-      <state_interface name="position"/>
+      <state_interface name="position">
+        <param name="initial_value">-2.00</param>
+      </state_interface>
       <state_interface name="velocity"/>
       <state_interface name="effort"/>
@@ -97,5 +107,7 @@
     <joint name="left_revolute_1">
       <command_interface name="effort"/>
-      <state_interface name="position"/>
+      <state_interface name="position">
+        <param name="initial_value">-1.53</param>
+      </state_interface>
       <state_interface name="velocity"/>
       <state_interface name="effort"/>
@@ -103,5 +115,7 @@
     <joint name="left_revolute_2">
       <command_interface name="effort"/>
-      <state_interface name="position"/>
+      <state_interface name="position">
+        <param name="initial_value">-2.82</param>
+      </state_interface>
       <state_interface name="velocity"/>
       <state_interface name="effort"/>
@@ -109,5 +123,7 @@
     <joint name="left_revolute_3">
       <command_interface name="effort"/>
-      <state_interface name="position"/>
+      <state_interface name="position">
+        <param name="initial_value">-2.00</param>
+      </state_interface>
       <state_interface name="velocity"/>
       <state_interface name="effort"/>

File: exo_right_arm_ws/src/exo_description/urdf/exo_arm_left.xacro (robot description, xacro)
@@ -1,5 +1,5 @@
 <?xml version="1.0" ?>
 <robot name="exo_arm_left" xmlns:xacro="http://www.ros.org/wiki/xacro">
-<xacro:macro name="exo_arm_left" params="prefix mount_x mount_y mount_z mount_roll mount_pitch mount_yaw">
+<xacro:macro name="exo_arm_left" params="prefix mount_x mount_y mount_z mount_roll mount_pitch mount_yaw joint_dynamics:=false">
 <xacro:property name="arm_base_link" value="${prefix + 'base_link' if prefix != '' else 'base_link'}"/>
 <xacro:if value="${prefix != ''}">
@@ -12,7 +12,7 @@
 <link name="${arm_base_link}">
   <inertial>
-    <origin xyz="-0.06548033561011322 -3.616267163486952e-05 -0.024681014225333156" rpy="0 0 0"/>
+    <origin xyz="-0.06508829102930236 -0.0016392947082375286 -0.029106797642733048" rpy="0 0 0"/>
     <mass value="0.071076"/>
-    <inertia ixx="0.00057" iyy="0.001116" izz="0.000764" ixy="3e-06" iyz="6.9e-05" ixz="-0.000381"/>
+    <inertia ixx="0.000253" iyy="0.00039" izz="0.000225" ixy="-9e-06" iyz="-4e-06" ixz="-0.000127"/>
   </inertial>
   <visual>
@@ -23,4 +23,5 @@
     <material name="silver"/>
   </visual>
+  <xacro:if value="${joint_dynamics}">
   <collision>
     <origin xyz="0 0 0" rpy="0 0 0"/>
@@ -29,13 +30,14 @@
     </geometry>
   </collision>
+  </xacro:if>
 </link>
 <link name="${prefix}motor_1">
   <inertial>
-    <origin xyz="-0.028657149518970373 8.058698600191602e-05 -0.0008100661993833275" rpy="0 0 0"/>
-    <mass value="0.33655768521614"/>
-    <inertia ixx="0.000158" iyy="0.000208" izz="0.000206" ixy="0.0" iyz="-0.0" ixz="-7e-06"/>
-  </inertial>
-  <visual>
-    <origin xyz="0.093353 -0.0 0.038143" rpy="0 0 0"/>
+    <origin xyz="-0.028657148535228882 -0.0008037659584219806 0.00012366679922792834" rpy="0 0 0"/>
+    <mass value="0.3365576984957861"/>
+    <inertia ixx="0.000158" iyy="0.000207" izz="0.000208" ixy="-7e-06" iyz="1e-06" ixz="1e-06"/>
+  </inertial>
+  <visual>
+    <origin xyz="0.094353 -0.00061 0.063136" rpy="0 0 0"/>
     <geometry>
       <mesh filename="package://exo_description/meshes/exo_assembly/left/Left_Motor_1_1.stl" scale="0.001 0.001 0.001"/>
@@ -43,19 +45,21 @@
     <material name="silver"/>
   </visual>
-  <collision>
-    <origin xyz="0.093353 -0.0 0.038143" rpy="0 0 0"/>
+  <xacro:if value="${joint_dynamics}">
+  <collision>
+    <origin xyz="0.094353 -0.00061 0.063136" rpy="0 0 0"/>
     <geometry>
       <mesh filename="package://exo_description/meshes/exo_assembly/left/Left_Motor_1_1.stl" scale="0.001 0.001 0.001"/>
     </geometry>
   </collision>
+  </xacro:if>
 </link>
 <link name="${prefix}component_1">
   <inertial>
-    <origin xyz="0.02007815411342466 0.07680678650680861 0.00015979042048477887" rpy="0 0 0"/>
-    <mass value="0.103407"/>
-    <inertia ixx="0.0015" iyy="0.001127" izz="0.002243" ixy="-0.000743" iyz="-2.8e-05" ixz="-5.2e-05"/>
-  </inertial>
-  <visual>
-    <origin xyz="0.096353 -0.0 0.038143" rpy="0 0 0"/>
+    <origin xyz="0.017291080002229037 0.002735639742798342 0.08182000531860147" rpy="0 0 0"/>
+    <mass value="0.13580987071810816"/>
+    <inertia ixx="0.000224" iyy="0.000337" izz="0.000165" ixy="4e-06" iyz="-2e-06" ixz="-0.000101"/>
+  </inertial>
+  <visual>
+    <origin xyz="0.097353 -0.00061 0.063136" rpy="0 0 0"/>
     <geometry>
       <mesh filename="package://exo_description/meshes/exo_assembly/left/Left_Component_1_1.stl" scale="0.001 0.001 0.001"/>
@@ -63,19 +67,21 @@
     <material name="silver"/>
   </visual>
-  <collision>
-    <origin xyz="0.096353 -0.0 0.038143" rpy="0 0 0"/>
+  <xacro:if value="${joint_dynamics}">
+  <collision>
+    <origin xyz="0.097353 -0.00061 0.063136" rpy="0 0 0"/>
     <geometry>
       <mesh filename="package://exo_description/meshes/exo_assembly/left/Left_Component_1_1.stl" scale="0.001 0.001 0.001"/>
     </geometry>
   </collision>
+  </xacro:if>
 </link>
 <link name="${prefix}motor_2">
   <inertial>
-    <origin xyz="0.0008094176185517183 0.025656899220221727 8.018870374155301e-05" rpy="0 0 0"/>
-    <mass value="0.33655768521614"/>
-    <inertia ixx="0.000206" iyy="0.000158" izz="0.000208" ixy="-7e-06" iyz="-0.0" ixz="0.0"/>
-  </inertial>
-  <visual>
-    <origin xyz="0.009353 -0.107 0.038143" rpy="0 0 0"/>
+    <origin xyz="9.522009318585489e-05 8.756209107413371e-05 0.025669346895594282" rpy="0 0 0"/>
+    <mass value="0.3365576984957861"/>
+    <inertia ixx="0.000208" iyy="0.000207" izz="0.000158" ixy="0.0" iyz="5e-06" ixz="-1e-06"/>
+  </inertial>
+  <visual>
+    <origin xyz="0.010353 -0.004345 -0.043799" rpy="0 0 0"/>
     <geometry>
       <mesh filename="package://exo_description/meshes/exo_assembly/left/Left_Motor_2_1.stl" scale="0.001 0.001 0.001"/>
@@ -83,19 +89,21 @@
     <material name="silver"/>
   </visual>
-  <collision>
-    <origin xyz="0.009353 -0.107 0.038143" rpy="0 0 0"/>
+  <xacro:if value="${joint_dynamics}">
+  <collision>
+    <origin xyz="0.010353 -0.004345 -0.043799" rpy="0 0 0"/>
     <geometry>
       <mesh filename="package://exo_description/meshes/exo_assembly/left/Left_Motor_2_1.stl" scale="0.001 0.001 0.001"/>
     </geometry>
   </collision>
+  </xacro:if>
 </link>
 <link name="${prefix}component_2">
   <inertial>
-    <origin xyz="1.739567280411962e-05 -0.0065127043001018264 -0.06684120565439666" rpy="0 0 0"/>
-    <mass value="0.069014"/>
-    <inertia ixx="0.001293" iyy="0.001346" izz="6.3e-05" ixy="0.0" iyz="-1e-06" ixz="0.0"/>
-  </inertial>
-  <visual>
-    <origin xyz="0.009353 -0.104 0.038143" rpy="0 0 0"/>
+    <origin xyz="0.02130252609513996 -0.06354392139822984 -0.004297968633705511" rpy="0 0 0"/>
+    <mass value="0.06901401596668413"/>
+    <inertia ixx="0.000158" iyy="2.6e-05" izz="0.000182" ixy="5e-05" iyz="5e-06" ixz="-2e-06"/>
+  </inertial>
+  <visual>
+    <origin xyz="0.010353 -0.00424 -0.040801" rpy="0 0 0"/>
     <geometry>
       <mesh filename="package://exo_description/meshes/exo_assembly/left/Left_Component_2_1.stl" scale="0.001 0.001 0.001"/>
@@ -103,19 +111,21 @@
     <material name="silver"/>
   </visual>
-  <collision>
-    <origin xyz="0.009353 -0.104 0.038143" rpy="0 0 0"/>
+  <xacro:if value="${joint_dynamics}">
+  <collision>
+    <origin xyz="0.010353 -0.00424 -0.040801" rpy="0 0 0"/>
     <geometry>
       <mesh filename="package://exo_description/meshes/exo_assembly/left/Left_Component_2_1.stl" scale="0.001 0.001 0.001"/>
     </geometry>
   </collision>
+  </xacro:if>
 </link>
 <link name="${prefix}component_3">
   <inertial>
-    <origin xyz="-0.0062448498075838264 -0.023063684617812677 -0.09933411008225428" rpy="0 0 0"/>
-    <mass value="0.276754"/>
-    <inertia ixx="0.009623" iyy="0.00994" izz="0.001914" ixy="-0.0003" iyz="0.00023" ixz="-0.000599"/>
-  </inertial>
-  <visual>
-    <origin xyz="0.009341 -0.103 0.083713" rpy="0 0 0"/>
+    <origin xyz="0.03615700401627118 -0.08448867239925995 -0.008977979556696391" rpy="0 0 0"/>
+    <mass value="0.25726311190565365"/>
+    <inertia ixx="0.001177" iyy="0.000369" izz="0.001416" ixy="0.0004" iyz="2.1e-05" ixz="3.6e-05"/>
+  </inertial>
+  <visual>
+    <origin xyz="-0.007995 0.050713 -0.030712" rpy="0 0 0"/>
     <geometry>
       <mesh filename="package://exo_description/meshes/exo_assembly/left/Left_Component_3_1.stl" scale="0.001 0.001 0.001"/>
@@ -123,19 +133,21 @@
     <material name="silver"/>
   </visual>
-  <collision>
-    <origin xyz="0.009341 -0.103 0.083713" rpy="0 0 0"/>
+  <xacro:if value="${joint_dynamics}">
+  <collision>
+    <origin xyz="-0.007995 0.050713 -0.030712" rpy="0 0 0"/>
     <geometry>
       <mesh filename="package://exo_description/meshes/exo_assembly/left/Left_Component_3_1.stl" scale="0.001 0.001 0.001"/>
     </geometry>
   </collision>
+  </xacro:if>
 </link>
 <link name="${prefix}motor_3">
   <inertial>
-    <origin xyz="-0.0005186558966796062 0.02813050113080831 0.00550509151078743" rpy="0 0 0"/>
-    <mass value="0.33655768521614"/>
-    <inertia ixx="0.000208" iyy="0.000161" izz="0.000203" ixy="4e-06" iyz="-1.3e-05" ixz="1e-06"/>
-  </inertial>
-  <visual>
-    <origin xyz="0.007241 -0.11298 0.328465" rpy="0 0 0"/>
+    <origin xyz="-0.0002717727838932593 0.00017757175027499628 0.028666777586146615" rpy="0 0 0"/>
+    <mass value="0.3365576984957861"/>
+    <inertia ixx="0.000208" iyy="0.000207" izz="0.000158" ixy="-0.0" iyz="5e-06" ixz="2e-06"/>
+  </inertial>
+  <visual>
+    <origin xyz="-0.07979 0.264928 -0.040288" rpy="0 0 0"/>
     <geometry>
       <mesh filename="package://exo_description/meshes/exo_assembly/left/Left_Motor_3_1.stl" scale="0.001 0.001 0.001"/>
@@ -143,19 +155,21 @@
     <material name="silver"/>
   </visual>
-  <collision>
-    <origin xyz="0.007241 -0.11298 0.328465" rpy="0 0 0"/>
+  <xacro:if value="${joint_dynamics}">
+  <collision>
+    <origin xyz="-0.07979 0.264928 -0.040288" rpy="0 0 0"/>
     <geometry>
       <mesh filename="package://exo_description/meshes/exo_assembly/left/Left_Motor_3_1.stl" scale="0.001 0.001 0.001"/>
     </geometry>
   </collision>
+  </xacro:if>
 </link>
 <link name="${prefix}component_4">
   <inertial>
-    <origin xyz="-0.004872320231196634 0.005488292975636799 -0.08462064279454101" rpy="0 0 0"/>
-    <mass value="0.070944"/>
-    <inertia ixx="0.001503" iyy="0.00162" izz="0.000292" ixy="-8.6e-05" iyz="7.5e-05" ixz="-3.2e-05"/>
-  </inertial>
-  <visual>
-    <origin xyz="0.00724 -0.115936 0.327953" rpy="0 0 0"/>
+    <origin xyz="-0.08439620971621951 0.0033097944704012505 -0.008999385990610932" rpy="0 0 0"/>
+    <mass value="0.07092471532695957"/>
+    <inertia ixx="4.2e-05" iyy="0.000201" izz="0.000218" ixy="1.3e-05" iyz="-1e-05" ixz="-2.2e-05"/>
+  </inertial>
+  <visual>
+    <origin xyz="-0.079795 0.264831 -0.043287" rpy="0 0 0"/>
     <geometry>
       <mesh filename="package://exo_description/meshes/exo_assembly/left/Left_Component_4_1.stl" scale="0.001 0.001 0.001"/>
@@ -163,18 +177,22 @@
     <material name="silver"/>
   </visual>
-  <collision>
-    <origin xyz="0.00724 -0.115936 0.327953" rpy="0 0 0"/>
+  <xacro:if value="${joint_dynamics}">
+  <collision>
+    <origin xyz="-0.079795 0.264831 -0.043287" rpy="0 0 0"/>
     <geometry>
       <mesh filename="package://exo_description/meshes/exo_assembly/left/Left_Component_4_1.stl" scale="0.001 0.001 0.001"/>
     </geometry>
   </collision>
+  </xacro:if>
 </link>
 <joint name="${prefix}revolute_1" type="revolute">
-  <origin xyz="-0.093353 0.0 -0.038143" rpy="0 0 0"/>
+  <origin xyz="-0.094353 0.00061 -0.063136" rpy="0 0 0"/>
   <parent link="${arm_base_link}"/>
   <child link="${prefix}motor_1"/>
   <axis xyz="1.0 0.0 0.0"/>
+  <xacro:if value="${joint_dynamics}">
   <dynamics damping="0.012" friction="0.1184"/>
-  <limit lower="0" upper="1.919" effort="20" velocity="11"/>
+  </xacro:if>
+  <limit lower="-3.14" upper="0" effort="20" velocity="11"/>
 </joint>
 <joint name="${prefix}fixed_1" type="fixed">
@@ -184,31 +202,35 @@
 </joint>
 <joint name="${prefix}fixed_2" type="fixed">
-  <origin xyz="0.087 0.107 0.0" rpy="0 0 0"/>
+  <origin xyz="0.087 0.003735 0.106935" rpy="0 0 0"/>
   <parent link="${prefix}component_1"/>
   <child link="${prefix}motor_2"/>
 </joint>
 <joint name="${prefix}revolute_2" type="revolute">
-  <origin xyz="0.0 -0.003 0.0" rpy="0 0 0"/>
+  <origin xyz="0.0 -0.000105 -0.002998" rpy="0 0 0"/>
   <parent link="${prefix}motor_2"/>
   <child link="${prefix}component_2"/>
-  <axis xyz="-0.0 -1.0 0.0"/>
+  <axis xyz="0.0 -0.034899 -0.999391"/>
+  <xacro:if value="${joint_dynamics}">
   <dynamics damping="0.012" friction="0.1184"/>
-  <limit lower="-0.56" upper="2.793" effort="20" velocity="11"/>
+  </xacro:if>
+  <limit lower="-3.3" upper="0" effort="20" velocity="11"/>
 </joint>
 <joint name="${prefix}fixed_3" type="fixed">
-  <origin xyz="1.2e-05 -0.001 -0.04557" rpy="0 0 0"/>
+  <origin xyz="0.018348 -0.054953 -0.010089" rpy="0 0 0"/>
   <parent link="${prefix}component_2"/>
   <child link="${prefix}component_3"/>
 </joint>
 <joint name="${prefix}revolute_3" type="revolute">
-  <origin xyz="0.0021 0.00998 -0.244752" rpy="0 0 0"/>
+  <origin xyz="0.071795 -0.214215 0.009576" rpy="0 0 0"/>
   <parent link="${prefix}component_3"/>
   <child link="${prefix}motor_3"/>
-  <axis xyz="-7.9e-05 -0.985338 -0.170613"/>
+  <axis xyz="-0.001694 -0.032292 -0.999477"/>
+  <xacro:if value="${joint_dynamics}">
   <dynamics damping="0.012" friction="0.1184"/>
-  <limit lower="0" upper="2.094" effort="20" velocity="11"/>
+  </xacro:if>
+  <limit lower="-2.08" upper="0" effort="20" velocity="11"/>
 </joint>
 <joint name="${prefix}fixed_4" type="fixed">
-  <origin xyz="1e-06 0.002956 0.000512" rpy="0 0 0"/>
+  <origin xyz="5e-06 9.7e-05 0.002999" rpy="0 0 0"/>
   <parent link="${prefix}motor_3"/>
   <child link="${prefix}component_4"/>
