Commit message: exo_description update and smc tuning

File: exo_right_arm_ws/src/exo_description/urdf/exo_arm_right.xacro (robot description, xacro)
@@ -1,5 +1,5 @@
 <?xml version="1.0" ?>
 <robot name="exo_arm_right" xmlns:xacro="http://www.ros.org/wiki/xacro">
-<xacro:macro name="exo_arm_right" params="prefix mount_x mount_y mount_z mount_roll mount_pitch mount_yaw">
+<xacro:macro name="exo_arm_right" params="prefix mount_x mount_y mount_z mount_roll mount_pitch mount_yaw joint_dynamics:=false">
 <xacro:property name="arm_base_link" value="${prefix + 'base_link' if prefix != '' else 'base_link'}"/>
 <xacro:if value="${prefix != ''}">
@@ -12,7 +12,7 @@
 <link name="${arm_base_link}">
   <inertial>
-    <origin xyz="-0.06548033529530813 3.6162664937364756e-05 -0.024681013869616315" rpy="0 0 0"/>
+    <origin xyz="-0.06508828909321891 0.0016392932839860918 -0.029106794021422928" rpy="0 0 0"/>
     <mass value="0.071076"/>
-    <inertia ixx="0.00057" iyy="0.001116" izz="0.000764" ixy="-3e-06" iyz="-6.9e-05" ixz="-0.000381"/>
+    <inertia ixx="0.000208" iyy="0.00032" izz="0.000185" ixy="8e-06" iyz="3e-06" ixz="-0.000104"/>
   </inertial>
   <visual>
@@ -23,4 +23,5 @@
     <material name="silver"/>
   </visual>
+  <xacro:if value="${joint_dynamics}">
   <collision>
     <origin xyz="0 0 0" rpy="0 0 0"/>
@@ -29,13 +30,14 @@
     </geometry>
   </collision>
+  </xacro:if>
 </link>
 <link name="${prefix}component_1">
   <inertial>
-    <origin xyz="0.020078154117980904 -0.07680678655412938 0.00015979036369085514" rpy="0 0 0"/>
-    <mass value="0.103407"/>
-    <inertia ixx="0.0015" iyy="0.001127" izz="0.002243" ixy="0.000743" iyz="2.8e-05" ixz="-5.2e-05"/>
-  </inertial>
-  <visual>
-    <origin xyz="0.096353 0.0 0.038143" rpy="0 0 0"/>
+    <origin xyz="0.020078156586478324 -0.002520887276899919 0.07676564491860602" rpy="0 0 0"/>
+    <mass value="0.10340048966459635"/>
+    <inertia ixx="0.000203" iyy="0.000303" izz="0.000152" ixy="-4e-06" iyz="1e-06" ixz="-0.0001"/>
+  </inertial>
+  <visual>
+    <origin xyz="0.097353 0.00061 0.063136" rpy="0 0 0"/>
     <geometry>
       <mesh filename="package://exo_description/meshes/exo_assembly/right/Right_Component_1_1.stl" scale="0.001 0.001 0.001"/>
@@ -43,19 +45,21 @@
     <material name="silver"/>
   </visual>
-  <collision>
-    <origin xyz="0.096353 0.0 0.038143" rpy="0 0 0"/>
+  <xacro:if value="${joint_dynamics}">
+  <collision>
+    <origin xyz="0.097353 0.00061 0.063136" rpy="0 0 0"/>
     <geometry>
       <mesh filename="package://exo_description/meshes/exo_assembly/right/Right_Component_1_1.stl" scale="0.001 0.001 0.001"/>
     </geometry>
   </collision>
+  </xacro:if>
 </link>
 <link name="${prefix}motor_1">
   <inertial>
-    <origin xyz="-0.028657149296548154 -8.058668921841178e-05 -0.000810066210235709" rpy="0 0 0"/>
-    <mass value="0.33655768070512687"/>
-    <inertia ixx="0.000158" iyy="0.000208" izz="0.000206" ixy="-0.0" iyz="0.0" ixz="-7e-06"/>
-  </inertial>
-  <visual>
-    <origin xyz="0.093353 0.0 0.038143" rpy="0 0 0"/>
+    <origin xyz="-0.028657146735079228 -0.0008124469950160578 5.2337020642223564e-05" rpy="0 0 0"/>
+    <mass value="0.33655768070512676"/>
+    <inertia ixx="0.000158" iyy="0.000206" izz="0.000208" ixy="-7e-06" iyz="-0.0" ixz="0.0"/>
+  </inertial>
+  <visual>
+    <origin xyz="0.094353 0.00061 0.063136" rpy="0 0 0"/>
     <geometry>
       <mesh filename="package://exo_description/meshes/exo_assembly/right/Right_Motor_1_1.stl" scale="0.001 0.001 0.001"/>
@@ -63,19 +67,21 @@
     <material name="silver"/>
   </visual>
-  <collision>
-    <origin xyz="0.093353 0.0 0.038143" rpy="0 0 0"/>
+  <xacro:if value="${joint_dynamics}">
+  <collision>
+    <origin xyz="0.094353 0.00061 0.063136" rpy="0 0 0"/>
     <geometry>
       <mesh filename="package://exo_description/meshes/exo_assembly/right/Right_Motor_1_1.stl" scale="0.001 0.001 0.001"/>
     </geometry>
   </collision>
+  </xacro:if>
 </link>
 <link name="${prefix}motor_2">
   <inertial>
-    <origin xyz="0.0008094176294007934 -0.02565689899779973 8.018840696268764e-05" rpy="0 0 0"/>
-    <mass value="0.33655768070512687"/>
-    <inertia ixx="0.000206" iyy="0.000158" izz="0.000208" ixy="7e-06" iyz="0.0" ixz="0.0"/>
-  </inertial>
-  <visual>
-    <origin xyz="0.009353 0.107 0.038143" rpy="0 0 0"/>
+    <origin xyz="0.0008094200168279157 -0.0008145820388575867 0.02564395698733552" rpy="0 0 0"/>
+    <mass value="0.33655768070512676"/>
+    <inertia ixx="0.000206" iyy="0.000208" izz="0.000158" ixy="0.0" iyz="1e-06" ixz="-7e-06"/>
+  </inertial>
+  <visual>
+    <origin xyz="0.010353 0.004345 -0.043799" rpy="0 0 0"/>
     <geometry>
       <mesh filename="package://exo_description/meshes/exo_assembly/right/Right_Motor_2_1.stl" scale="0.001 0.001 0.001"/>
@@ -83,19 +89,21 @@
     <material name="silver"/>
   </visual>
-  <collision>
-    <origin xyz="0.009353 0.107 0.038143" rpy="0 0 0"/>
+  <xacro:if value="${joint_dynamics}">
+  <collision>
+    <origin xyz="0.010353 0.004345 -0.043799" rpy="0 0 0"/>
     <geometry>
       <mesh filename="package://exo_description/meshes/exo_assembly/right/Right_Motor_2_1.stl" scale="0.001 0.001 0.001"/>
     </geometry>
   </collision>
+  </xacro:if>
 </link>
 <link name="${prefix}component_2">
   <inertial>
-    <origin xyz="1.7395672801560902e-05 0.006512704300103006 -0.06684120565439672" rpy="0 0 0"/>
-    <mass value="0.069014"/>
-    <inertia ixx="0.001293" iyy="0.001346" izz="6.3e-05" ixy="-0.0" iyz="1e-06" ixz="0.0"/>
-  </inertial>
-  <visual>
-    <origin xyz="0.009353 0.104 0.038143" rpy="0 0 0"/>
+    <origin xyz="0.02170967506266145 0.06340564193577251 -0.004302798150324916" rpy="0 0 0"/>
+    <mass value="0.06901401423488361"/>
+    <inertia ixx="0.000157" iyy="2.6e-05" izz="0.000182" ixy="-5.1e-05" iyz="-5e-06" ixz="-2e-06"/>
+  </inertial>
+  <visual>
+    <origin xyz="0.010353 0.00424 -0.040801" rpy="0 0 0"/>
     <geometry>
       <mesh filename="package://exo_description/meshes/exo_assembly/right/Right_Component_2_1.stl" scale="0.001 0.001 0.001"/>
@@ -103,19 +111,21 @@
     <material name="silver"/>
   </visual>
-  <collision>
-    <origin xyz="0.009353 0.104 0.038143" rpy="0 0 0"/>
+  <xacro:if value="${joint_dynamics}">
+  <collision>
+    <origin xyz="0.010353 0.00424 -0.040801" rpy="0 0 0"/>
     <geometry>
       <mesh filename="package://exo_description/meshes/exo_assembly/right/Right_Component_2_1.stl" scale="0.001 0.001 0.001"/>
     </geometry>
   </collision>
+  </xacro:if>
 </link>
 <link name="${prefix}component_3">
   <inertial>
-    <origin xyz="-0.00624485437452308 0.023063684861781966 -0.09933410970644764" rpy="0 0 0"/>
-    <mass value="0.276754"/>
-    <inertia ixx="0.009623" iyy="0.00994" izz="0.001914" ixy="0.0003" iyz="-0.00023" ixz="-0.000599"/>
-  </inertial>
-  <visual>
-    <origin xyz="0.009341 0.092 0.083713" rpy="0 0 0"/>
+    <origin xyz="0.0362007475571462 0.08488733536574525 -0.02097339196773956" rpy="0 0 0"/>
+    <mass value="0.2572924347231441"/>
+    <inertia ixx="0.001177" iyy="0.00037" izz="0.001416" ixy="-0.0004" iyz="-2.1e-05" ixz="3.6e-05"/>
+  </inertial>
+  <visual>
+    <origin xyz="-0.008346 -0.050211 -0.041702" rpy="0 0 0"/>
     <geometry>
       <mesh filename="package://exo_description/meshes/exo_assembly/right/Right_Component_3_1.stl" scale="0.001 0.001 0.001"/>
@@ -123,19 +133,21 @@
     <material name="silver"/>
   </visual>
-  <collision>
-    <origin xyz="0.009341 0.092 0.083713" rpy="0 0 0"/>
+  <xacro:if value="${joint_dynamics}">
+  <collision>
+    <origin xyz="-0.008346 -0.050211 -0.041702" rpy="0 0 0"/>
     <geometry>
       <mesh filename="package://exo_description/meshes/exo_assembly/right/Right_Component_3_1.stl" scale="0.001 0.001 0.001"/>
     </geometry>
   </collision>
+  </xacro:if>
 </link>
 <link name="${prefix}motor_3">
   <inertial>
-    <origin xyz="0.0005239633876655348 -0.028343595073468772 0.004273928835601515" rpy="0 0 0"/>
-    <mass value="0.33655768070512687"/>
-    <inertia ixx="0.000208" iyy="0.000158" izz="0.000207" ixy="4e-06" iyz="3e-06" ixz="-0.0"/>
-  </inertial>
-  <visual>
-    <origin xyz="0.007241 0.10198 0.328465" rpy="0 0 0"/>
+    <origin xyz="0.00071319645679499 -0.0004566132738064721 0.028656360017304303" rpy="0 0 0"/>
+    <mass value="0.33655768070512676"/>
+    <inertia ixx="0.000207" iyy="0.000208" izz="0.000158" ixy="-0.0" iyz="-2e-06" ixz="-6e-06"/>
+  </inertial>
+  <visual>
+    <origin xyz="-0.080242 -0.26481 -0.039283" rpy="0 0 0"/>
     <geometry>
       <mesh filename="package://exo_description/meshes/exo_assembly/right/Right_Motor_3_1.stl" scale="0.001 0.001 0.001"/>
@@ -143,19 +155,21 @@
     <material name="silver"/>
   </visual>
-  <collision>
-    <origin xyz="0.007241 0.10198 0.328465" rpy="0 0 0"/>
+  <xacro:if value="${joint_dynamics}">
+  <collision>
+    <origin xyz="-0.080242 -0.26481 -0.039283" rpy="0 0 0"/>
     <geometry>
       <mesh filename="package://exo_description/meshes/exo_assembly/right/Right_Motor_3_1.stl" scale="0.001 0.001 0.001"/>
     </geometry>
   </collision>
+  </xacro:if>
 </link>
 <link name="${prefix}component_4">
   <inertial>
-    <origin xyz="-0.0048723202311687815 -0.005488292975653827 -0.08462064279554748" rpy="0 0 0"/>
-    <mass value="0.070944"/>
-    <inertia ixx="0.001503" iyy="0.00162" izz="0.000292" ixy="8.6e-05" iyz="-7.5e-05" ixz="-3.2e-05"/>
-  </inertial>
-  <visual>
-    <origin xyz="0.00724 0.104936 0.327953" rpy="0 0 0"/>
+    <origin xyz="-0.08441969431975782 -0.002715032580566934 -0.008979759026676165" rpy="0 0 0"/>
+    <mass value="0.07092471532503089"/>
+    <inertia ixx="4.2e-05" iyy="0.000201" izz="0.000218" ixy="-1.2e-05" iyz="1e-05" ixz="-2.2e-05"/>
+  </inertial>
+  <visual>
+    <origin xyz="-0.080247 -0.264713 -0.042282" rpy="0 0 0"/>
     <geometry>
       <mesh filename="package://exo_description/meshes/exo_assembly/right/Right_Component_4_1.stl" scale="0.001 0.001 0.001"/>
@@ -163,10 +177,12 @@
     <material name="silver"/>
   </visual>
-  <collision>
-    <origin xyz="0.00724 0.104936 0.327953" rpy="0 0 0"/>
+  <xacro:if value="${joint_dynamics}">
+  <collision>
+    <origin xyz="-0.080247 -0.264713 -0.042282" rpy="0 0 0"/>
     <geometry>
       <mesh filename="package://exo_description/meshes/exo_assembly/right/Right_Component_4_1.stl" scale="0.001 0.001 0.001"/>
     </geometry>
   </collision>
+  </xacro:if>
 </link>
 <joint name="${prefix}fixed_1" type="fixed">
@@ -176,39 +192,45 @@
 </joint>
 <joint name="${prefix}revolute_1" type="revolute">
-  <origin xyz="-0.093353 0.0 -0.038143" rpy="0 0 0"/>
+  <origin xyz="-0.094353 -0.00061 -0.063136" rpy="0 0 0"/>
   <parent link="${arm_base_link}"/>
   <child link="${prefix}motor_1"/>
   <axis xyz="-1.0 -0.0 0.0"/>
+  <xacro:if value="${joint_dynamics}">
   <dynamics damping="0.012" friction="0.1184"/>
-  <limit lower="0" upper="1.919" effort="20" velocity="11"/>
+  </xacro:if>
+  <limit lower="-3.14" upper="0" effort="20" velocity="11"/>
 </joint>
 <joint name="${prefix}fixed_2" type="fixed">
-  <origin xyz="0.087 -0.107 0.0" rpy="0 0 0"/>
+  <origin xyz="0.087 -0.003735 0.106935" rpy="0 0 0"/>
   <parent link="${prefix}component_1"/>
   <child link="${prefix}motor_2"/>
 </joint>
 <joint name="${prefix}revolute_2" type="revolute">
-  <origin xyz="0.0 0.003 0.0" rpy="0 0 0"/>
+  <origin xyz="0.0 0.000105 -0.002998" rpy="0 0 0"/>
   <parent link="${prefix}motor_2"/>
   <child link="${prefix}component_2"/>
-  <axis xyz="0.0 -1.0 0.0"/>
+  <axis xyz="0.0 -0.034899 0.999391"/>
+  <xacro:if value="${joint_dynamics}">
   <dynamics damping="0.012" friction="0.1184"/>
-  <limit lower="-0.56" upper="2.793" effort="20" velocity="11"/>
+  </xacro:if>
+  <limit lower="-3.3" upper="0" effort="20" velocity="11"/>
 </joint>
 <joint name="${prefix}fixed_3" type="fixed">
-  <origin xyz="1.2e-05 0.012 -0.04557" rpy="0 0 0"/>
+  <origin xyz="0.018699 0.054451 0.000901" rpy="0 0 0"/>
   <parent link="${prefix}component_2"/>
   <child link="${prefix}component_3"/>
 </joint>
 <joint name="${prefix}revolute_3" type="revolute">
-  <origin xyz="0.0021 -0.00998 -0.244752" rpy="0 0 0"/>
+  <origin xyz="0.071896 0.214599 -0.002419" rpy="0 0 0"/>
   <parent link="${prefix}component_3"/>
   <child link="${prefix}motor_3"/>
-  <axis xyz="7.9e-05 -0.985338 0.170613"/>
+  <axis xyz="0.001695 -0.032293 0.999477"/>
+  <xacro:if value="${joint_dynamics}">
   <dynamics damping="0.012" friction="0.1184"/>
-  <limit lower="0" upper="2.094" effort="20" velocity="11"/>
+  </xacro:if>
+  <limit lower="-2.08" upper="0" effort="20" velocity="11"/>
 </joint>
 <joint name="${prefix}fixed_4" type="fixed">
-  <origin xyz="1e-06 -0.002956 0.000512" rpy="0 0 0"/>
+  <origin xyz="5e-06 -9.7e-05 0.002999" rpy="0 0 0"/>
   <parent link="${prefix}motor_3"/>
   <child link="${prefix}component_4"/>

Commit message: added mass disturbances option

File: exo_right_arm_ws/src/exo_description/urdf/exo.xacro (robot description, xacro)
@@ -22,4 +22,20 @@
 <xacro:arg name="left_mount_pitch" default="0"/>
 <xacro:arg name="left_mount_yaw" default="0"/>
+<!-- Simulation-only mass disturbances. Defaults are 0, and the pre-built dynamics
+     URDFs used by model-based controllers are generated without these args, so the
+     controllers' dynamic model never sees them. Only the gazebo launch propagates
+     non-zero values. -->
+<xacro:arg name="right_extra_mass_component_1" default="0"/>
+<xacro:arg name="right_extra_mass_component_2" default="0"/>
+<xacro:arg name="right_extra_mass_component_3" default="0"/>
+<xacro:arg name="right_extra_mass_component_4" default="0"/>
+<xacro:arg name="right_payload_mass" default="0"/>
+<xacro:arg name="left_extra_mass_component_1" default="0"/>
+<xacro:arg name="left_extra_mass_component_2" default="0"/>
+<xacro:arg name="left_extra_mass_component_3" default="0"/>
+<xacro:arg name="left_extra_mass_component_4" default="0"/>
+<xacro:arg name="left_payload_mass" default="0"/>
+<!-- Shared radius [m] for the spherical inertia model of every extra mass. -->
+<xacro:arg name="extra_mass_radius" default="0.05"/>
 <xacro:include filename="$(find exo_description)/urdf/materials.xacro" />
 <xacro:include filename="$(find exo_description)/urdf/exo_arm_right.xacro" />
@@ -43,5 +59,11 @@
     mount_x="${xacro.arg('right_mount_x')}" mount_y="${xacro.arg('right_mount_y')}" mount_z="${xacro.arg('right_mount_z')}"
     mount_roll="${xacro.arg('right_mount_roll')}" mount_pitch="${xacro.arg('right_mount_pitch')}" mount_yaw="${xacro.arg('right_mount_yaw')}"
-    joint_dynamics="${xacro.arg('joint_dynamics')}"/>
+    joint_dynamics="${xacro.arg('joint_dynamics')}"
+    m_extra_component_1="${xacro.arg('right_extra_mass_component_1')}"
+    m_extra_component_2="${xacro.arg('right_extra_mass_component_2')}"
+    m_extra_component_3="${xacro.arg('right_extra_mass_component_3')}"
+    m_extra_component_4="${xacro.arg('right_extra_mass_component_4')}"
+    m_payload="${xacro.arg('right_payload_mass')}"
+    extra_mass_radius="${xacro.arg('extra_mass_radius')}"/>
 </xacro:if>
 <xacro:if value="${xacro.arg('arms') == 'dual' or xacro.arg('arms') == 'left'}">
@@ -49,5 +71,11 @@
     mount_x="${xacro.arg('left_mount_x')}" mount_y="${xacro.arg('left_mount_y')}" mount_z="${xacro.arg('left_mount_z')}"
     mount_roll="${xacro.arg('left_mount_roll')}" mount_pitch="${xacro.arg('left_mount_pitch')}" mount_yaw="${xacro.arg('left_mount_yaw')}"
-    joint_dynamics="${xacro.arg('joint_dynamics')}"/>
+    joint_dynamics="${xacro.arg('joint_dynamics')}"
+    m_extra_component_1="${xacro.arg('left_extra_mass_component_1')}"
+    m_extra_component_2="${xacro.arg('left_extra_mass_component_2')}"
+    m_extra_component_3="${xacro.arg('left_extra_mass_component_3')}"
+    m_extra_component_4="${xacro.arg('left_extra_mass_component_4')}"
+    m_payload="${xacro.arg('left_payload_mass')}"
+    extra_mass_radius="${xacro.arg('extra_mass_radius')}"/>
 </xacro:if>
 <ros2_control name="exo_system" type="system">

File: exo_right_arm_ws/src/exo_description/urdf/exo_arm_left.xacro (robot description, xacro)
@@ -1,6 +1,15 @@
 <?xml version="1.0" ?>
 <robot name="exo_arm_left" xmlns:xacro="http://www.ros.org/wiki/xacro">
-<xacro:macro name="exo_arm_left" params="prefix mount_x mount_y mount_z mount_roll mount_pitch mount_yaw joint_dynamics:=false">
+<xacro:macro name="exo_arm_left" params="prefix mount_x mount_y mount_z mount_roll mount_pitch mount_yaw joint_dynamics:=false
+  m_extra_component_1:=0 m_extra_component_2:=0 m_extra_component_3:=0 m_extra_component_4:=0 m_payload:=0
+  extra_mass_radius:=0.05">
 <xacro:property name="arm_base_link" value="${prefix + 'base_link' if prefix != '' else 'base_link'}"/>
+<!-- Each extra mass is modeled as a uniform solid sphere centered at the link's
+     existing COM; contribution to ixx/iyy/izz is (2/5)*m*r^2. Off-diagonals are
+     unaffected because the sphere is symmetric about the same COM. -->
+<xacro:property name="_di_c1" value="${0.4 * m_extra_component_1 * extra_mass_radius * extra_mass_radius}"/>
+<xacro:property name="_di_c2" value="${0.4 * m_extra_component_2 * extra_mass_radius * extra_mass_radius}"/>
+<xacro:property name="_di_c3" value="${0.4 * m_extra_component_3 * extra_mass_radius * extra_mass_radius}"/>
+<xacro:property name="_di_c4" value="${0.4 * (m_extra_component_4 + m_payload) * extra_mass_radius * extra_mass_radius}"/>
 <xacro:if value="${prefix != ''}">
   <joint name="${prefix}mount_joint" type="fixed">
@@ -57,6 +66,6 @@
   <inertial>
     <origin xyz="0.017291080002229037 0.002735639742798342 0.08182000531860147" rpy="0 0 0"/>
-    <mass value="0.13580987071810816"/>
-    <inertia ixx="0.000224" iyy="0.000337" izz="0.000165" ixy="4e-06" iyz="-2e-06" ixz="-0.000101"/>
+    <mass value="${0.13580987071810816 + m_extra_component_1}"/>
+    <inertia ixx="${0.000224 + _di_c1}" iyy="${0.000337 + _di_c1}" izz="${0.000165 + _di_c1}" ixy="4e-06" iyz="-2e-06" ixz="-0.000101"/>
   </inertial>
   <visual>
@@ -101,6 +110,6 @@
   <inertial>
     <origin xyz="0.02130252609513996 -0.06354392139822984 -0.004297968633705511" rpy="0 0 0"/>
-    <mass value="0.06901401596668413"/>
-    <inertia ixx="0.000158" iyy="2.6e-05" izz="0.000182" ixy="5e-05" iyz="5e-06" ixz="-2e-06"/>
+    <mass value="${0.06901401596668413 + m_extra_component_2}"/>
+    <inertia ixx="${0.000158 + _di_c2}" iyy="${2.6e-05 + _di_c2}" izz="${0.000182 + _di_c2}" ixy="5e-05" iyz="5e-06" ixz="-2e-06"/>
   </inertial>
   <visual>
@@ -123,6 +132,6 @@
   <inertial>
     <origin xyz="0.03615700401627118 -0.08448867239925995 -0.008977979556696391" rpy="0 0 0"/>
-    <mass value="0.25726311190565365"/>
-    <inertia ixx="0.001177" iyy="0.000369" izz="0.001416" ixy="0.0004" iyz="2.1e-05" ixz="3.6e-05"/>
+    <mass value="${0.25726311190565365 + m_extra_component_3}"/>
+    <inertia ixx="${0.001177 + _di_c3}" iyy="${0.000369 + _di_c3}" izz="${0.001416 + _di_c3}" ixy="0.0004" iyz="2.1e-05" ixz="3.6e-05"/>
   </inertial>
   <visual>
@@ -167,6 +176,6 @@
   <inertial>
     <origin xyz="-0.08439620971621951 0.0033097944704012505 -0.008999385990610932" rpy="0 0 0"/>
-    <mass value="0.07092471532695957"/>
-    <inertia ixx="4.2e-05" iyy="0.000201" izz="0.000218" ixy="1.3e-05" iyz="-1e-05" ixz="-2.2e-05"/>
+    <mass value="${0.07092471532695957 + m_extra_component_4 + m_payload}"/>
+    <inertia ixx="${4.2e-05 + _di_c4}" iyy="${0.000201 + _di_c4}" izz="${0.000218 + _di_c4}" ixy="1.3e-05" iyz="-1e-05" ixz="-2.2e-05"/>
   </inertial>
   <visual>

File: exo_right_arm_ws/src/exo_description/urdf/exo_arm_right.xacro (robot description, xacro)
@@ -1,6 +1,15 @@
 <?xml version="1.0" ?>
 <robot name="exo_arm_right" xmlns:xacro="http://www.ros.org/wiki/xacro">
-<xacro:macro name="exo_arm_right" params="prefix mount_x mount_y mount_z mount_roll mount_pitch mount_yaw joint_dynamics:=false">
+<xacro:macro name="exo_arm_right" params="prefix mount_x mount_y mount_z mount_roll mount_pitch mount_yaw joint_dynamics:=false
+  m_extra_component_1:=0 m_extra_component_2:=0 m_extra_component_3:=0 m_extra_component_4:=0 m_payload:=0
+  extra_mass_radius:=0.05">
 <xacro:property name="arm_base_link" value="${prefix + 'base_link' if prefix != '' else 'base_link'}"/>
+<!-- Each extra mass is modeled as a uniform solid sphere centered at the link's
+     existing COM; contribution to ixx/iyy/izz is (2/5)*m*r^2. Off-diagonals are
+     unaffected because the sphere is symmetric about the same COM. -->
+<xacro:property name="_di_c1" value="${0.4 * m_extra_component_1 * extra_mass_radius * extra_mass_radius}"/>
+<xacro:property name="_di_c2" value="${0.4 * m_extra_component_2 * extra_mass_radius * extra_mass_radius}"/>
+<xacro:property name="_di_c3" value="${0.4 * m_extra_component_3 * extra_mass_radius * extra_mass_radius}"/>
+<xacro:property name="_di_c4" value="${0.4 * (m_extra_component_4 + m_payload) * extra_mass_radius * extra_mass_radius}"/>
 <xacro:if value="${prefix != ''}">
   <joint name="${prefix}mount_joint" type="fixed">
@@ -35,6 +44,6 @@
   <inertial>
     <origin xyz="0.020078156586478324 -0.002520887276899919 0.07676564491860602" rpy="0 0 0"/>
-    <mass value="0.10340048966459635"/>
-    <inertia ixx="0.000203" iyy="0.000303" izz="0.000152" ixy="-4e-06" iyz="1e-06" ixz="-0.0001"/>
+    <mass value="${0.10340048966459635 + m_extra_component_1}"/>
+    <inertia ixx="${0.000203 + _di_c1}" iyy="${0.000303 + _di_c1}" izz="${0.000152 + _di_c1}" ixy="-4e-06" iyz="1e-06" ixz="-0.0001"/>
   </inertial>
   <visual>
@@ -101,6 +110,6 @@
   <inertial>
     <origin xyz="0.02170967506266145 0.06340564193577251 -0.004302798150324916" rpy="0 0 0"/>
-    <mass value="0.06901401423488361"/>
-    <inertia ixx="0.000157" iyy="2.6e-05" izz="0.000182" ixy="-5.1e-05" iyz="-5e-06" ixz="-2e-06"/>
+    <mass value="${0.06901401423488361 + m_extra_component_2}"/>
+    <inertia ixx="${0.000157 + _di_c2}" iyy="${2.6e-05 + _di_c2}" izz="${0.000182 + _di_c2}" ixy="-5.1e-05" iyz="-5e-06" ixz="-2e-06"/>
   </inertial>
   <visual>
@@ -123,6 +132,6 @@
   <inertial>
     <origin xyz="0.0362007475571462 0.08488733536574525 -0.02097339196773956" rpy="0 0 0"/>
-    <mass value="0.2572924347231441"/>
-    <inertia ixx="0.001177" iyy="0.00037" izz="0.001416" ixy="-0.0004" iyz="-2.1e-05" ixz="3.6e-05"/>
+    <mass value="${0.2572924347231441 + m_extra_component_3}"/>
+    <inertia ixx="${0.001177 + _di_c3}" iyy="${0.00037 + _di_c3}" izz="${0.001416 + _di_c3}" ixy="-0.0004" iyz="-2.1e-05" ixz="3.6e-05"/>
   </inertial>
   <visual>
@@ -167,6 +176,6 @@
   <inertial>
     <origin xyz="-0.08441969431975782 -0.002715032580566934 -0.008979759026676165" rpy="0 0 0"/>
-    <mass value="0.07092471532503089"/>
-    <inertia ixx="4.2e-05" iyy="0.000201" izz="0.000218" ixy="-1.2e-05" iyz="1e-05" ixz="-2.2e-05"/>
+    <mass value="${0.07092471532503089 + m_extra_component_4 + m_payload}"/>
+    <inertia ixx="${4.2e-05 + _di_c4}" iyy="${0.000201 + _di_c4}" izz="${0.000218 + _di_c4}" ixy="-1.2e-05" iyz="1e-05" ixz="-2.2e-05"/>
   </inertial>
   <visual>
