Commit message: implemented forward kinematics

File: exo_right_arm_ws/src/exo_description/urdf/exo.xacro (robot description, xacro)
@@ -110,5 +110,5 @@
       <command_interface name="effort"/>
       <state_interface name="position">
-        <param name="initial_value">-1.53</param>
+        <param name="initial_value">0</param>
       </state_interface>
       <state_interface name="velocity"/>
@@ -118,5 +118,5 @@
       <command_interface name="effort"/>
       <state_interface name="position">
-        <param name="initial_value">-2.82</param>
+        <param name="initial_value">0</param>
       </state_interface>
       <state_interface name="velocity"/>
@@ -126,5 +126,5 @@
       <command_interface name="effort"/>
       <state_interface name="position">
-        <param name="initial_value">-2.00</param>
+        <param name="initial_value">0</param>
       </state_interface>
       <state_interface name="velocity"/>
@@ -136,5 +136,5 @@
       <command_interface name="effort"/>
       <state_interface name="position">
-        <param name="initial_value">-1.53</param>
+        <param name="initial_value">0</param>
       </state_interface>
       <state_interface name="velocity"/>
@@ -144,5 +144,5 @@
       <command_interface name="effort"/>
       <state_interface name="position">
-        <param name="initial_value">-2.82</param>
+        <param name="initial_value">0</param>
       </state_interface>
       <state_interface name="velocity"/>
@@ -152,5 +152,5 @@
       <command_interface name="effort"/>
       <state_interface name="position">
-        <param name="initial_value">-2.00</param>
+        <param name="initial_value">0</param>
       </state_interface>
       <state_interface name="velocity"/>

File: exo_right_arm_ws/src/exo_description/urdf/exo_arm_left.xacro (robot description, xacro)
@@ -196,5 +196,5 @@
 </link>
 <joint name="${prefix}revolute_1" type="revolute">
-  <origin xyz="-0.094353 0.00061 -0.063136" rpy="0 0 0"/>
+  <origin xyz="-0.094353 0.00061 -0.063136" rpy="-1.5358897 0 0"/>
   <parent link="${arm_base_link}"/>
   <child link="${prefix}motor_1"/>
@@ -203,5 +203,5 @@
   <dynamics damping="0.012" friction="0.1184"/>
   </xacro:if>
-  <limit lower="-3.14" upper="0" effort="20" velocity="11"/>
+  <limit lower="-1.6041" upper="1.5359" effort="20" velocity="11"/>
 </joint>
 <joint name="${prefix}fixed_1" type="fixed">
@@ -216,5 +216,5 @@
 </joint>
 <joint name="${prefix}revolute_2" type="revolute">
-  <origin xyz="0.0 -0.000105 -0.002998" rpy="0 0 0"/>
+  <origin xyz="0.0 -0.000105 -0.002998" rpy="0.0679119 0.0113622 2.8101676"/>
   <parent link="${prefix}motor_2"/>
   <child link="${prefix}component_2"/>
@@ -223,5 +223,5 @@
   <dynamics damping="0.012" friction="0.1184"/>
   </xacro:if>
-  <limit lower="-3.3" upper="0" effort="20" velocity="11"/>
+  <limit lower="-0.4900" upper="2.8100" effort="20" velocity="11"/>
 </joint>
 <joint name="${prefix}fixed_3" type="fixed">
@@ -231,5 +231,5 @@
 </joint>
 <joint name="${prefix}revolute_3" type="revolute">
-  <origin xyz="0.071795 -0.214215 0.009576" rpy="0 0 0"/>
+  <origin xyz="0.071795 -0.214215 0.009576" rpy="0.0499166 0.0254288 2.0945769"/>
   <parent link="${prefix}component_3"/>
   <child link="${prefix}motor_3"/>
@@ -238,5 +238,5 @@
   <dynamics damping="0.012" friction="0.1184"/>
   </xacro:if>
-  <limit lower="-2.08" upper="0" effort="20" velocity="11"/>
+  <limit lower="0" upper="2.0944" effort="20" velocity="11"/>
 </joint>
 <joint name="${prefix}fixed_4" type="fixed">

File: exo_right_arm_ws/src/exo_description/urdf/exo_arm_right.xacro (robot description, xacro)
@@ -201,12 +201,12 @@
 </joint>
 <joint name="${prefix}revolute_1" type="revolute">
-  <origin xyz="-0.094353 -0.00061 -0.063136" rpy="0 0 0"/>
+  <origin xyz="-0.094353 -0.00061 -0.063136" rpy="1.5358897 0 0"/>
   <parent link="${arm_base_link}"/>
   <child link="${prefix}motor_1"/>
-  <axis xyz="-1.0 -0.0 0.0"/>
+  <axis xyz="-1.0 0.0 0.0"/>
   <xacro:if value="${joint_dynamics}">
   <dynamics damping="0.012" friction="0.1184"/>
   </xacro:if>
-  <limit lower="-3.14" upper="0" effort="20" velocity="11"/>
+  <limit lower="-1.6041" upper="1.5359" effort="20" velocity="11"/>
 </joint>
 <joint name="${prefix}fixed_2" type="fixed">
@@ -216,5 +216,5 @@
 </joint>
 <joint name="${prefix}revolute_2" type="revolute">
-  <origin xyz="0.0 0.000105 -0.002998" rpy="0 0 0"/>
+  <origin xyz="0.0 0.000105 -0.002998" rpy="-0.0679119 0.0113622 -2.8101676"/>
   <parent link="${prefix}motor_2"/>
   <child link="${prefix}component_2"/>
@@ -223,5 +223,5 @@
   <dynamics damping="0.012" friction="0.1184"/>
   </xacro:if>
-  <limit lower="-3.3" upper="0" effort="20" velocity="11"/>
+  <limit lower="-0.4900" upper="2.8100" effort="20" velocity="11"/>
 </joint>
 <joint name="${prefix}fixed_3" type="fixed">
@@ -231,5 +231,5 @@
 </joint>
 <joint name="${prefix}revolute_3" type="revolute">
-  <origin xyz="0.071896 0.214599 -0.002419" rpy="0 0 0"/>
+  <origin xyz="0.071896 0.214599 -0.002419" rpy="-0.0499189 0.0254281 -2.0945768"/>
   <parent link="${prefix}component_3"/>
   <child link="${prefix}motor_3"/>
@@ -238,5 +238,5 @@
   <dynamics damping="0.012" friction="0.1184"/>
   </xacro:if>
-  <limit lower="-2.08" upper="0" effort="20" velocity="11"/>
+  <limit lower="0" upper="2.0944" effort="20" velocity="11"/>
 </joint>
 <joint name="${prefix}fixed_4" type="fixed">
